File: KiCad/IBM_5324_Keyboard.kicad_sch (KiCad schematic)
At the start: 84 parts, among them SW1 CMD, SW10 ERASE, SW11 1!, SW12 3#, SW13 5%, SW14 7&, SW15 +*, SW16 9(, SW17 -_, SW18 +*, SW19 -/, SW2 `~, SW20 NP_8, SW21 HOLD, SW22 FIELD ADV, SW23 W, SW24 R, SW25 Y, SW26 I, SW27 P, SW28 \|, SW29 NP_7, SW3 2@, SW30 NP_9, SW31 INQ, SW32 CAPS LOCK, SW33 Q, SW34 E, SW35 T, SW36 O, SW37 !¢, SW38 ENTER, SW39 NP_4, SW4 4$, SW40 FIELD-, SW41 U, SW42 ERROR RESET, SW43 SHIFT, SW44 A, SW45 D, SW46 G, SW47 J, SW48 L, SW49 '", SW5 6^, SW50 {}, SW51 NP_5, SW52 NP_6, SW53 TEST, SW54 SCROLL DOWN, SW55 S, SW56 F, SW57 H, SW58 SCROLL UP, SW59 K, SW6 8*, SW60 ;:, SW61 NEWLINE, SW62 NP_1, SW63 NP_3, SW64 ->, SW65 <>, SW66 C, SW67 B, SW68 M, SW69 ., SW7 0), SW70 RH_SHIFT, SW71 NP_2, SW72 FIELD+, SW73 N, SW74 <-, SW75 ALT, SW76 Z, SW77 X, SW78 V, SW79 SPACE, SW8 =+, SW80 ,, SW81 /?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

Commit message: Finalise keyboard matrix layout
Parts:
- removed SW9: <-, symbol Switch:SW_Push_45deg
- SW11: value 1! -> | 1
- SW12: value 3# -> # 3
- SW13: value 5% -> % 5
- SW14: value 7& -> & 7
- SW15: value +* -> * +
- SW16: value 9( -> ( 9
- SW17: value -_ -> _ -
- SW18: value +* -> RH <-
- SW19: value -/ -> / -
- SW2: value `~ -> ~ `
- SW20: value NP_8 -> NP 8
- SW28: value \| -> | \
- SW29: value NP_7 -> NP 7
- SW3: value 2@ -> @ 2
- SW30: value NP_9 -> NP 9
- SW32: value CAPS LOCK -> SHIFT LOCK
- SW37: value !¢ -> ! ¢
- SW39: value NP_4 -> NP 4
- SW4: value 4$ -> $ 4
- SW43: value SHIFT -> LH SHIFT
- SW49: value '" -> " '
- SW5: value 6^ -> ^ 6
- SW50: value {} -> } {
- SW51: value NP_5 -> NP 5
- SW52: value NP_6 -> NP 6
- SW6: value 8* -> * 8
- SW60: value ;: -> : ;
- SW62: value NP_1 -> NP 1
- SW63: value NP_3 -> NP 3
- SW65: value <> -> > <
- SW69: value . -> . .
- SW7: value 0) -> ) 0
- SW70: value RH_SHIFT -> RH SHIFT
- SW71: value NP_2 -> NP 2
- SW74: value <- -> LH <-
- SW8: value =+ -> + =
- SW80: value , -> , ,
- SW81: value /? -> ? /
- SW83: value NP_0 -> NP 0
- SW84: value NP_. -> NP .

Commit message: PCB layout started
Parts:
- added KB1: SPACE, PCM_Mounting_Keyboard_Stabilizer:Stabilizer_Cherry_MX_8.00u, symbol Clueless_Engineer:Stabiliser
- added KB2: FIELD+, PCM_Mounting_Keyboard_Stabilizer:Stabilizer_Cherry_MX_3.00u, symbol Clueless_Engineer:Stabiliser
- SW1, SW10, SW11, SW12, SW13, SW14, SW16, SW17, SW18, SW2, SW20, SW21, SW23, SW24, SW25, SW26, SW27, SW28, SW29, SW3, SW30, SW31, SW33, SW34, SW35, SW36, SW37, SW39, SW4, SW40, SW41, SW42, SW44, SW45, SW46, SW47, SW48, SW49, SW5, SW50, SW51, SW52, SW53, SW54, SW55, SW56, SW57, SW58, SW59, SW6, SW60, SW61, SW62, SW63, SW64, SW66, SW67, SW68, SW69, SW7, SW71, SW73, SW74, SW76, SW77, SW78, SW79, SW8, SW80, SW81: footprint (none) -> PCM_Switch_Keyboard_Cherry_MX:SW_Cherry_MX_PCB
- SW15, SW19, SW32: footprint (none) -> PCM_Switch_Keyboard_Cherry_MX:SW_Cherry_MX_PCB_1.75u
- SW22, SW70: footprint (none) -> PCM_Switch_Keyboard_Cherry_MX:SW_Cherry_MX_PCB_1.50u
- SW38: footprint (none) -> PCM_Switch_Keyboard_Cherry_MX:SW_Cherry_MX_PCB_2.00u_90deg
- SW43: footprint (none) -> PCM_Switch_Keyboard_Cherry_MX:SW_Cherry_MX_PCB_1.25u
- SW65: footprint (none) -> PCM_Switch_Keyboard_Cherry_MX:SW_Cherry_MX_PCB_1.00u
- SW72: footprint (none) -> PCM_Switch_Keyboard_Cherry_MX:SW_Cherry_MX_PCB_3.00u_90deg
- SW75: footprint (none) -> PCM_Switch_Keyboard_Cherry_MX:SW_Cherry_MX_PCB_2.25u
- SW82, SW83, SW84: footprint (none) -> PCM_Switch_Keyboard_Cherry_MX:SW_Cherry_MX_PCB_2.00u
Other:
- moved on the sheet: SW1, SW10, SW11, SW12, SW13, SW14, SW15, SW16, SW17, SW18, SW19, SW2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
