File: KiCad/IBM_5324_Keyboard.kicad_sch (KiCad schematic)
At the start: 107 parts, among them J1 To 5324, J2 To DB25, SW1 CMD, SW10 ERASE, SW11 | 1, SW12 # 3, SW13 % 5, SW14 & 7, SW15 ( 9, SW16 _ -, SW17 RH <-, SW18 NP 8, SW19 / -, SW2 ~ `, SW20 HOLD, SW21 FIELD ADV, SW22 W, SW23 R, SW24 Y, SW25 I, SW26 P, SW27 | \, SW28 NP 7, SW29 NP 9, SW3 @ 2, SW30 INQ, SW31 SHIFT LOCK, SW32 Q, SW33 E, SW34 T, SW35 U, SW36 O, SW37 ! ¢, SW38 ENTER, SW39 NP 4, SW4 $ 4, SW40 FIELD-, SW41 ERROR RESET, SW42 LH SHIFT, SW43 A, SW44 D, SW45 G, SW46 J, SW47 L, SW48 " ', SW49 } {, SW5 ^ 6, SW50 NP 5, SW51 NP 6, SW52 TEST, SW53 SCROLL DOWN, SW54 S, SW55 F, SW56 H, SW57 K, SW58 : ;, SW59 NEWLINE, SW6 * 8, SW60 NP 1, SW61 NP 3, SW62 SCROLL UP, SW63 ->, SW64 > <, SW65 C, SW66 B, SW67 N, SW68 M, SW69 . ., SW7 ) 0, SW70 RH SHIFT, SW71 NP 2, SW72 FIELD+, SW73 LH <-, SW74 ALT, SW75 Z, SW76 X, SW77 V, SW78 SPACE, SW79 , ,, SW8 + =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

Commit message: Added USB-B socket for Teensy programming/debugging
Parts:
- added J3: USB_B, Connector_USB:USB_B_Lumberg_2411_02_Horizontal, symbol Connector:USB_B
Connections:
- net GND: now also J3.4 (GND), J3.5 (Shield)
- net USB D-: now reaches U1.66 (D-)
- net USB D-: now also J3.2 (D-)
- net USB D+: now reaches U1.67 (D+)
- net USB D+: now also J3.3 (D+)
- net Col_A renamed COL A
- net Col_B renamed COL B
- net Col_C renamed COL C
- net Col_D renamed COL D
- net Col_E renamed COL E
- net Col_F renamed COL F
- net Col_G renamed COL G
- net Col_H renamed COL H
- net Col_I renamed COL I
- net Col_J renamed COL J
- net Col_K renamed COL K
- net Row_1 renamed ROW 1
- net Row_2 renamed ROW 2
- net Row_3 renamed ROW 3
- net Row_4 renamed ROW 4
- net Row_5 renamed ROW 5
- net Row_6 renamed ROW 6
- net Row_7 renamed ROW 7
- net Row_8 renamed ROW 8
- no-connect marks 38 -> 37
Other:
- note added: "2x14 pin header interface to DB25 cable."
- note added: "Additional USB port on motherboard for programming/debugging Teensy (optional, requires removal of USB-C on Teensy)."
- note added: "Buffered signals from host 5324."
- note added: "DB25 male interface to host 5324 via DB25 female-male extension cable."
- note added: "No Key"
- note added: "Not needed, opt for Teensy 4.1 without Ethernet if practical."
- note added: "Output signals to host 5324 are buffered to ensure logic highs are accurately read by the 5324. Input signals are similarly buffered."
- note added: "Spare gates left disabled."
- note added: "Unbuffered signals to host 5324."
- note removed: "2x14 pin header interface to DB25 cable"
- note removed: "Buffered signals from 5324"
- note removed: "DB25 male interface to 5324 via DB25 female-male extension cable."
- note removed: "Output signals to 5324 are buffered to ensure logic highs are accurately read by the 5324. Input signals are similarly buffered."
- note removed: "Spare gates left disabled"
- note removed: "Unbuffered signals to 5324"
