File: KiCad/IBM_5324_Keyboard.kicad_pcb (KiCad board)
At the start: 2 copper layers, 431 x 134 mm, 97 parts, among them J1 To 5324, J2 To DB25, SW1 CMD, SW10 ERASE, SW11 | 1, SW12 # 3, SW13 % 5, SW14 & 7, SW15 * +, SW16 ( 9, SW17 _ -, SW18 RH <-, SW19 / -, SW2 ~ `, SW20 NP 8, SW21 HOLD, SW22 FIELD ADV, SW23 W, SW24 R, SW25 Y, SW26 I, SW27 P, SW28 | \, SW29 NP 7, SW3 @ 2, SW30 NP 9, SW31 INQ, SW32 SHIFT LOCK, SW33 Q, SW34 E, SW35 T, SW36 O, SW37 ! ¢, SW38 ENTER, SW39 NP 4, SW4 $ 4, SW40 FIELD-, SW41 U, SW42 ERROR RESET, SW43 LH SHIFT, SW44 A, SW45 D, SW46 G, SW47 J, SW48 L, SW49 " ', SW5 ^ 6, SW50 } {, SW51 NP 5, SW52 NP 6, SW53 TEST, SW54 SCROLL DOWN, SW55 S, SW56 F, SW57 H, SW58 SCROLL UP, SW59 K, SW6 * 8, SW60 : ;, SW61 NEWLINE, SW62 NP 1, SW63 NP 3, SW64 ->, SW65 > <, SW66 C, SW67 B, SW68 M, SW69 . ., SW7 ) 0, SW70 RH SHIFT, SW71 NP 2, SW72 FIELD+, SW73 N, SW74 LH <-, SW75 ALT, SW76 Z, SW77 X, SW78 V, SW79 SPACE, SW8 + =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

Commit message: Initial layout completed
Parts:
- added C1: 10µF, Capacitor_THT:CP_Radial_D5.0mm_P2.50mm, F.Cu at (415.0, 181.0)
- added U3: 74HCT245, Package_DIP:DIP-18_W7.62mm, F.Cu at (420.1, 160.6)
- J2: footprint Connector_PinHeader_2.54mm:PinHeader_2x08_P2.54mm_Vertical -> Connector_PinHeader_2.54mm:PinHeader_2x14_P2.54mm_Vertical
- U2: value LM7805_TO220 -> TSR 2-2450; footprint Package_TO_SOT_THT:TO-220-3_Horizontal_TabDown -> Converter_DCDC:Converter_DCDC_TRACO_TSR2-24xxN_TSR2-24xxxN_THT
- moved U2 18.2 mm to (488.6, 181.0)
- moved J2 5.09 mm to (442.9, 181.0)
Connections:
- J1 pad 1: DATA STROBE -> DATA STROBE_{BUFF}
- J1 pad 2: SCAN CODE BIT 6 -> SCAN CODE BIT 6_{BUFF}
- J1 pad 3: SCAN CODE BIT 5 -> SCAN CODE BIT 5_{BUFF}
- J1 pad 4: SCAN CODE BIT 4 -> SCAN CODE BIT 4_{BUFF}
- J1 pad 5: SCAN CODE BIT 3 -> SCAN CODE BIT 3_{BUFF}
- J1 pad 6: SCAN CODE BIT 2 -> SCAN CODE BIT 2_{BUFF}
- J1 pad 7: SCAN CODE BIT 1 -> SCAN CODE BIT 1_{BUFF}
- J1 pad 8: SCAN CODE BIT 0 -> SCAN CODE BIT 0_{BUFF}
- J2 pad A1: unconnected-(J2-Pin_a1-PadA1) -> GND
- J2 pad A2: DELAY STROBE -> unconnected-(J2-PadA2)
- J2 pad A3: +12V -> GND
- J2 pad A4: unconnected-(J2-Pin_a4-PadA4) -> GND
- J2 pad A5: SCAN CODE BIT 0 -> GND
- J2 pad A6: unconnected-(J2-Pin_a6-PadA6) -> GND
- J2 pad A7: SCAN CODE BIT 1 -> GND
- J2 pad B1: PROGRAM RESET -> DATA STROBE_{BUFF}
- J2 pad B3: DATA STROBE -> SCAN CODE BIT 6_{BUFF}
- J2 pad B4: SCAN CODE BIT 6 -> SCAN CODE BIT 5_{BUFF}
- J2 pad B5: SCAN CODE BIT 5 -> SCAN CODE BIT 4_{BUFF}
- J2 pad B6: SCAN CODE BIT 4 -> SCAN CODE BIT 3_{BUFF}
- J2 pad B7: SCAN CODE BIT 3 -> SCAN CODE BIT 2_{BUFF}
- J2 pad B8: SCAN CODE BIT 2 -> SCAN CODE BIT 1_{BUFF}
- U1 pad 10: unconnected-(U1-8_TX2_IN1-Pad10) -> SCAN CODE BIT 6
- U1 pad 11: unconnected-(U1-9_OUT1C-Pad11) -> DATA STROBE
- U1 pad 12: unconnected-(U1-10_CS_MQSR-Pad12) -> DELAY STROBE
- U1 pad 13: unconnected-(U1-11_MOSI_CTX1-Pad13) -> PROGRAM RESET
- U1 pad 20: unconnected-(U1-28_RX7-Pad20) -> Col_E
- U1 pad 21: unconnected-(U1-29_TX7-Pad21) -> Col_D
- U1 pad 22: unconnected-(U1-30_CRX3-Pad22) -> Col_C
- U1 pad 23: unconnected-(U1-31_CTX3-Pad23) -> Col_B
- U1 pad 24: unconnected-(U1-32_OUT1B-Pad24) -> Col_A
- U1 pad 25: unconnected-(U1-33_MCLK2-Pad25) -> Col_F
- U1 pad 26: unconnected-(U1-34_RX8-Pad26) -> Col_G
- U1 pad 27: unconnected-(U1-35_TX8-Pad27) -> Col_H
- U1 pad 28: unconnected-(U1-36_CS-Pad28) -> Col_I
- U1 pad 29: unconnected-(U1-37_CS-Pad29) -> Col_J
- U1 pad 30: unconnected-(U1-38_CS1_IN1-Pad30) -> Col_K
- U1 pad 36: unconnected-(U1-14_A0_TX3_SPDIF_OUT-Pad36) -> Row_1
- U1 pad 37: unconnected-(U1-15_A1_RX3_SPDIF_IN-Pad37) -> Row_2
- U1 pad 38: unconnected-(U1-16_A2_RX4_SCL1-Pad38) -> Row_3
- U1 pad 39: unconnected-(U1-17_A3_TX4_SDA1-Pad39) -> Row_4
- U1 pad 4: unconnected-(U1-2_OUT2-Pad4) -> SCAN CODE BIT 0
- U1 pad 40: unconnected-(U1-18_A4_SDA-Pad40) -> Row_5
- U1 pad 41: unconnected-(U1-19_A5_SCL-Pad41) -> Row_6
- U1 pad 42: unconnected-(U1-20_A6_TX5_LRCLK1-Pad42) -> Row_7
- U1 pad 43: unconnected-(U1-21_A7_RX5_BCLK1-Pad43) -> Row_8
- U1 pad 5: unconnected-(U1-3_LRCLK2-Pad5) -> SCAN CODE BIT 1
- U1 pad 6: unconnected-(U1-4_BCLK2-Pad6) -> SCAN CODE BIT 2
- U1 pad 7: unconnected-(U1-5_IN2-Pad7) -> SCAN CODE BIT 3
- U1 pad 8: unconnected-(U1-6_OUT1D-Pad8) -> SCAN CODE BIT 4
- U1 pad 9: unconnected-(U1-7_RX2_OUT1A-Pad9) -> SCAN CODE BIT 5
Routing:
- net Col_A: track 133.4 -> 418.0 mm
- net Col_B: track 163.7 -> 374.6 mm
- net Row_8: track 404.0 -> 591.5 mm
- net Col_C: track 146.2 -> 321.6 mm
- net Row_6: track 393.9 -> 553.9 mm
- net Row_7: track 419.4 -> 571.7 mm
- net Row_5: track 400.3 -> 541.6 mm
- net Col_D: track 144.2 -> 284.1 mm
- net Row_3: track 366.5 -> 481.8 mm
- net Row_4: track 433.3 -> 545.1 mm
- net Col_K: track 122.2 -> 227.0 mm
- net Col_E: track 144.2 -> 248.5 mm
- net PROGRAM RESET: track 17.4 -> 103.9 mm
- net DELAY STROBE: track 12.8 -> 96.5 mm
- net Col_J: track 141.4 -> 210.9 mm
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Other:
- board text added: "A1 (ALL GROUND/RETURN THIS SIDE)"
- board text added: "B10"
- board text added: "B11"
- board text added: "B12"
- board text added: "B13"
- board text added: "B14"
- board text added: "B9"
- board text removed: "A1"
- board text removed: "A2"
- board text removed: "A3"
- board text removed: "A4"
- board text removed: "A5"
- board text removed: "A6"
- board text removed: "A7"
- board text removed: "A8"
