File: KiCad/IBM_5324_Keyboard.kicad_pcb (KiCad board)
At the start: 2 copper layers, 437 x 133 mm, 104 parts, among them J1 To 5324, J2 To DB25, SW1 CMD, SW10 ERASE, SW11 | 1, SW12 # 3, SW13 % 5, SW14 & 7, SW15 ( 9, SW16 _ -, SW17 RH <-, SW18 NP 8, SW19 / -, SW2 ~ `, SW20 HOLD, SW21 FIELD ADV, SW22 W, SW23 R, SW24 Y, SW25 I, SW26 P, SW27 | \, SW28 NP 7, SW29 NP 9, SW3 @ 2, SW30 INQ, SW31 SHIFT LOCK, SW32 Q, SW33 E, SW34 T, SW35 U, SW36 O, SW37 ! ¢, SW38 ENTER, SW39 NP 4, SW4 $ 4, SW40 FIELD-, SW41 ERROR RESET, SW42 LH SHIFT, SW43 A, SW44 D, SW45 G, SW46 J, SW47 L, SW48 " ', SW49 } {, SW5 ^ 6, SW50 NP 5, SW51 NP 6, SW52 TEST, SW53 SCROLL DOWN, SW54 S, SW55 F, SW56 H, SW57 K, SW58 : ;, SW59 NEWLINE, SW6 * 8, SW60 NP 1, SW61 NP 3, SW62 SCROLL UP, SW63 ->, SW64 > <, SW65 C, SW66 B, SW67 N, SW68 M, SW69 . ., SW7 ) 0, SW70 RH SHIFT, SW71 NP 2, SW72 FIELD+, SW73 LH <-, SW74 ALT, SW75 Z, SW76 X, SW77 V, SW78 SPACE, SW79 , ,, SW8 + =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

Commit message: Added 74LS125 buffer for incoming signals
Parts:
- added C2: 100nF, Capacitor_THT:C_Disc_D3.8mm_W2.6mm_P2.50mm, F.Cu at (411.2, 168.3)
- added C3: 100nF, Capacitor_THT:C_Disc_D3.8mm_W2.6mm_P2.50mm, F.Cu at (426.4, 160.6)
- added U4: 74HCT125, Package_DIP:DIP-14_W7.62mm, F.Cu at (399.7, 168.3)
- moved C1 50.8 mm to (351.5, 179.7)
- moved U2 42.1 mm to (373.1, 169.5), turned to 90 degrees
- moved RN1 28.2 mm to (390.9, 183.5), turned to 180 degrees
- moved D1 8.89 mm to (393.4, 160.6)
- moved D2 8.89 mm to (385.8, 160.6)
- moved R1 8.89 mm to (407.4, 164.5)
- moved R2 8.89 mm to (407.4, 160.6)
- moved U3 5.08 mm to (415.0, 160.6)
Connections:
- U1 pad 12: /PROGRAM RESET -> /PROGRAM RESE~{T}
- U1 pad 13: /DELAY STROBE -> /DELAY STROB~{E}
Routing:
- net /GND: track 0.00 -> 157.9 mm, vias 54 -> 19
- net /DELAY STROB~{E}: track 0.00 -> 114.8 mm
- net /DELAY STROBE: track 182.5 -> 69.6 mm, vias 0 -> 1
- net /PROGRAM RESE~{T}: track 0.00 -> 109.1 mm
- net /PROGRAM RESET: track 176.7 -> 73.5 mm, vias 0 -> 1
- net /+12V: track 63.5 -> 96.5 mm
- net /+5V: track 135.6 -> 150.0 mm
- net Row_2: track 523.9 -> 509.9 mm
- net Row_8: track 694.5 -> 681.7 mm
- net Row_7: track 672.9 -> 661.8 mm
- net Row_6: track 653.4 -> 644.0 mm
- net Row_1: track 434.3 -> 426.5 mm
- net Row_5: track 639.3 -> 631.7 mm
- net Row_4: track 641.0 -> 635.2 mm
- net /SCAN CODE BIT 6: track 55.9 -> 61.0 mm
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