File: KiCad/IBM_5324_Keyboard.kicad_pcb (KiCad board)
At the start: 2 copper layers, 437 x 133 mm, 107 parts, among them J1 To 5324, J2 To DB25, SW1 CMD, SW10 ERASE, SW11 | 1, SW12 # 3, SW13 % 5, SW14 & 7, SW15 ( 9, SW16 _ -, SW17 RH <-, SW18 NP 8, SW19 / -, SW2 ~ `, SW20 HOLD, SW21 FIELD ADV, SW22 W, SW23 R, SW24 Y, SW25 I, SW26 P, SW27 | \, SW28 NP 7, SW29 NP 9, SW3 @ 2, SW30 INQ, SW31 SHIFT LOCK, SW32 Q, SW33 E, SW34 T, SW35 U, SW36 O, SW37 ! ¢, SW38 ENTER, SW39 NP 4, SW4 $ 4, SW40 FIELD-, SW41 ERROR RESET, SW42 LH SHIFT, SW43 A, SW44 D, SW45 G, SW46 J, SW47 L, SW48 " ', SW49 } {, SW5 ^ 6, SW50 NP 5, SW51 NP 6, SW52 TEST, SW53 SCROLL DOWN, SW54 S, SW55 F, SW56 H, SW57 K, SW58 : ;, SW59 NEWLINE, SW6 * 8, SW60 NP 1, SW61 NP 3, SW62 SCROLL UP, SW63 ->, SW64 > <, SW65 C, SW66 B, SW67 N, SW68 M, SW69 . ., SW7 ) 0, SW70 RH SHIFT, SW71 NP 2, SW72 FIELD+, SW73 LH <-, SW74 ALT, SW75 Z, SW76 X, SW77 V, SW78 SPACE, SW79 , ,, SW8 + =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

Commit message: Added USB-B socket for Teensy programming/debugging
Parts:
- added J3: USB_B, Connector_USB:USB_B_Lumberg_2411_02_Horizontal, F.Cu at (227.8, 172.0)
Connections:
- U1 pad 66: unconnected-(U1-D--Pad66) -> /USB D-
- U1 pad 67: unconnected-(U1-D+-Pad67) -> /USB D+
Routing:
- net /GND: track 157.9 -> 1280.8 mm
- net /USB D-: track 0.00 -> 93.4 mm
- net /USB D+: track 0.00 -> 91.6 mm
Other:
- board text added: "Teensy USB Device (no power)"

Commit message: Reduced ground plane clearance to 0.3mm
Routing:
- net /GND: vias 42 -> 35
- net (no net): vias 1 -> 0
Changed lines of the file:
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@@
 		)
 	)
-	(via
-		(at 418.41765 123.181875)
-		(size 0.6)
-		(drill 0.3)
-		(layers "F.Cu" "B.Cu")
-		(net 0)
-	)
 	(segment
 		(start 244.80765 183.501875)
@@
 	)
 	(segment
+		(start 363.10765 177.191875)
+		(end 367.95765 177.191875)
+		(width 0.5)
+		(layer "F.Cu")
+		(net 21)
+	)
+	(segment
 		(start 367.95765 177.191875)
 		(end 375.61765 169.531875)
@@
 	(segment
 		(start 360.57765 177.191875)
-		(end 367.95765 177.191875)
+		(end 363.10765 177.191875)
 		(width 0.5)
 		(layer "F.Cu")
@@
 	)
 	(via
-		(at 401.48765 175.851875)
-		(size 0.6)
-		(drill 0.3)
-		(layers "F.Cu" "B.Cu")
-		(free yes)
-		(net 21)
-	)
-	(via
-		(at 404.62765 173.251875)
-		(size 0.6)
-		(drill 0.3)
-		(layers "F.Cu" "B.Cu")
-		(free yes)
-		(net 21)
-	)
-	(via
-		(at 396.56765 180.891875)
-		(size 0.6)
-		(drill 0.3)
-		(layers "F.Cu" "B.Cu")
-		(free yes)
-		(net 21)
-	)
-	(via
-		(at 448.83765 206.371875)
-		(size 0.6)
-		(drill 0.3)
-		(layers "F.Cu" "B.Cu")
-		(free yes)
-		(net 21)
-	)
-	(via
-		(at 409.79765 175.801875)
-		(size 0.6)
-		(drill 0.3)
-		(layers "F.Cu" "B.Cu")
-		(free yes)
-		(net 21)
-	)
-	(via
-		(at 344.32765 247.541875)
-		(size 0.6)
-		(drill 0.3)
-		(layers "F.Cu" "B.Cu")
-		(free yes)
-		(net 21)
-	)
-	(via
-		(at 404.62765 170.701875)
+		(at 282.10765 190.201875)
 		(size 0.6)
 		(drill 0.3)
@@
 	)
 	(via
-		(at 392.28765 175.781875)
+		(at 122.10765 268.451875)
 		(size 0.6)
 		(drill 0.3)
@@
 	)
 	(via
-		(at 404.62765 180.781875)
+		(at 378.35765 177.201875)
 		(size 0.6)
 		(drill 0.3)
@@
 	)
 	(via
-		(at 291.52765 223.851875)
+		(at 404.60765 180.701875)
 		(size 0.6)
 		(drill 0.3)
@@
 	)
 	(via
-		(at 272.95765 209.391875)
+		(at 234.85765 223.701875)
 		(size 0.6)
 		(drill 0.3)
@@
 	)
 	(via
-		(at 358.48765 190.441875)
+		(at 410.60765 173.201875)
 		(size 0.6)
 		(drill 0.3)
@@
 	)
 	(via
-		(at 397.22765 175.811875)
+		(at 404.60765 175.701875)
 		(size 0.6)
 		(drill 0.3)
@@
 	)
 	(via
-		(at 335.31765 177.201875)
+		(at 404.60765 178.701875)
 		(size 0.6)
 		(drill 0.3)
@@
 	)
 	(via
-		(at 121.41765 268.661875)
+		(at 396.85765 181.201875)
 		(size 0.6)
 		(drill 0.3)
@@
 	)
 	(via
-		(at 448.95765 258.531875)
+		(at 239.85765 171.951875)
 		(size 0.6)
 		(drill 0.3)
@@
 	)
 	(via
-		(at 379.47765 177.191875)
+		(at 163.60765 257.201875)
 		(size 0.6)
 		(drill 0.3)
@@
 	)
 	(via
-		(at 379.50765 171.501875)
+		(at 429.85765 242.951875)
 		(size 0.6)
 		(drill 0.3)
@@
 	)
 	(via
-		(at 163.63765 257.211875)
+		(at 429.85765 259.951875)
 		(size 0.6)
 		(drill 0.3)
@@
 	)
 	(via
-		(at 320.32765 202.681875)
+		(at 206.10765 190.701875)
 		(size 0.6)
 		(drill 0.3)
@@
 	)
 	(via
-		(at 277.58765 263.041875)
+		(at 310.60765 209.201875)
 		(size 0.6)
 		(drill 0.3)
@@
 	)
 	(via
-		(at 469.15765 222.501875)
+		(at 429.85765 222.951875)
 		(size 0.6)
 		(drill 0.3)
@@
 	)
 	(via
-		(at 397.25765 183.471875)
+		(at 396.85765 175.701875)
 		(size 0.6)
 		(drill 0.3)
@@
 	)
 	(via
-		(at 225.07765 192.061875)
+		(at 394.85765 178.701875)
 		(size 0.6)
 		(drill 0.3)
@@
 	)
 	(via
-		(at 272.62765 223.761875)
+		(at 472.85765 179.451875)
 		(size 0.6)
 		(drill 0.3)
@@
 	)
 	(via
-		(at 206.07765 190.661875)
+		(at 168.10765 190.701875)
 		(size 0.6)
 		(drill 0.3)
@@
 	)
 	(via
-		(at 404.62765 175.761875)
+		(at 404.60765 170.701875)
 		(size 0.6)
 		(drill 0.3)
@@
 	)
 	(via
-		(at 330.22765 222.941875)
+		(at 200.85765 228.701875)
 		(size 0.6)
 		(drill 0.3)
@@
 	)
 	(via
-		(at 411.78765 182.841875)
+		(at 358.10765 190.451875)
 		(size 0.6)
 		(drill 0.3)
@@
 	)
 	(via
-		(at 411.00765 178.801875)
+		(at 408.10765 190.701875)
 		(size 0.6)
 		(drill 0.3)
@@
 	)
 	(via
-		(at 167.86765 190.351875)
+		(at 448.85765 206.451875)
 		(size 0.6)
 		(drill 0.3)
@@
 	)
 	(via
-		(at 448.64765 242.851875)
+		(at 473.60765 218.451875)
 		(size 0.6)
 		(drill 0.3)
@@
 	)
 	(via
-		(at 196.20765 209.491875)
+		(at 348.60765 209.451875)
 		(size 0.6)
 		(drill 0.3)
@@
 	)
 	(via
-		(at 360.57765 177.191875)
-		(size 0.6)
-		(drill 0.3)
-		(layers "F.Cu" "B.Cu")
-		(net 21)
-	)
-	(via
-		(at 448.83765 223.951875)
+		(at 335.35765 177.201875)
 		(size 0.6)
 		(drill 0.3)
@@
 	)
 	(via
-		(at 408.17765 190.381875)
+		(at 310.60765 222.701875)
 		(size 0.6)
 		(drill 0.3)
@@
 	)
 	(via
-		(at 402.31765 183.601875)
+		(at 476.85765 240.451875)
 		(size 0.6)
 		(drill 0.3)
@@
 	)
 	(via
-		(at 477.39765 227.441875)
+		(at 368.60765 222.451875)
 		(size 0.6)
 		(drill 0.3)
@@
 	)
 	(via
-		(at 411.00765 172.911875)
+		(at 286.85765 262.951875)
 		(size 0.6)
 		(drill 0.3)
@@
 	)
 	(via
-		(at 394.15765 178.141875)
+		(at 320.10765 190.451875)
 		(size 0.6)
 		(drill 0.3)
@@
 	)
 	(via
-		(at 234.38765 209.491875)
+		(at 277.10765 228.451875)
 		(size 0.6)
 		(drill 0.3)
@@
 	)
 	(via
-		(at 404.62765 178.341875)
+		(at 363.10765 177.191875)
 		(size 0.6)
 		(drill 0.3)
 		(layers "F.Cu" "B.Cu")
-		(free yes)
 		(net 21)
 	)
@@
 	)
 	(via
-		(at 446.48765 184.141875)
+		(at 446.44765 184.101875)
 		(size 0.6)
 		(drill 0.3)
@@
 	)
 	(segment
+		(start 448.51765 185.191875)
+		(end 448.46765 185.191875)
+		(width 0.2)
+		(layer "B.Cu")
+		(net 33)
+	)
+	(segment
 		(start 450.09265 179.4402)
 		(end 450.09265 184.276875)
@@
 	(segment
 		(start 449.17765 185.191875)
-		(end 448.46765 185.191875)
+		(end 448.51765 185.191875)
 		(width 0.2)
 		(layer "B.Cu")
@@
 		(hatch edge 0.5)
 		(connect_pads
-			(clearance 0.5)
+			(clearance 0.3)
 		)
 		(min_thickness 0.25)
